File: ESP_01_5V.brd (EAGLE design)
At the start: 15.4 x 24.8 mm, 12 parts, among them IC1 REG1117, IC2 IC_TXB0108-TSSOP-20

Commit message: update
Parts:
- renumbered ESP01 to MOD1
Changed lines of the file:
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@@
 <attribute name="VALUE" x="3.8338125" y="19.796125" size="0.4064" layer="27" font="vector" rot="R180"/>
 </element>
-<element name="ESP01" library="esp8266modules" package="ESP01" value="ESP01" x="7.8978125" y="9.763125" smashed="yes" rot="MR0"/>
+<element name="MOD1" library="esp8266modules" package="ESP01" value="ESP01" x="7.8978125" y="9.763125" smashed="yes" rot="MR0"/>
 <element name="IC1" library="burr-brown" package="SOT223" value="REG1117" x="7.8184375" y="12.85875" smashed="yes" rot="R180">
 <attribute name="OC_NEWARK" value="14P6981" x="7.8184375" y="12.85875" size="1.778" layer="27" rot="R180" display="off"/>
@@
 <contactref element="C5" pad="1"/>
 <contactref element="JP1" pad="1"/>
-<contactref element="ESP01" pad="GND"/>
+<contactref element="MOD1" pad="GND"/>
 <contactref element="JP3" pad="2"/>
 <polygon width="0.4064" layer="16">
@@
 <contactref element="IC2" pad="3"/>
 <contactref element="C5" pad="2"/>
-<contactref element="ESP01" pad="VCC"/>
+<contactref element="MOD1" pad="VCC"/>
 <wire x1="7.62" y1="20.6375" x2="7.62" y2="19.685" width="0.254" layer="1"/>
 <wire x1="7.62" y1="19.685" x2="7.62" y2="18.7325" width="0.254" layer="1"/>
@@
 <signal name="N$9">
 <contactref element="JP2" pad="3"/>
-<contactref element="ESP01" pad="RST"/>
+<contactref element="MOD1" pad="RST"/>
 <wire x1="8.255" y1="3.175" x2="6.6675" y2="1.5875" width="0.254" layer="16"/>
 <wire x1="9.525" y1="3.175" x2="8.255" y2="3.175" width="0.254" layer="16"/>
@@
 <signal name="N$10">
 <contactref element="IC2" pad="7"/>
-<contactref element="ESP01" pad="RX"/>
+<contactref element="MOD1" pad="RX"/>
 <wire x1="6.6675" y1="5.08" x2="6.6675" y2="7.3025" width="0.254" layer="16"/>
 <wire x1="5.08" y1="5.08" x2="6.6675" y2="5.08" width="0.254" layer="16"/>
@@
 <signal name="N$11">
 <contactref element="IC2" pad="2"/>
-<contactref element="ESP01" pad="GPIO2"/>
+<contactref element="MOD1" pad="GPIO2"/>
 <wire x1="9.8425" y1="4.1275" x2="9.8425" y2="7.3025" width="0.254" layer="16"/>
 <wire x1="9.2075" y1="4.1275" x2="9.8425" y2="4.1275" width="0.254" layer="16"/>
@@
 <signal name="N$12">
 <contactref element="IC2" pad="4"/>
-<contactref element="ESP01" pad="GPIO0"/>
+<contactref element="MOD1" pad="GPIO0"/>
 <contactref element="JP3" pad="1"/>
 <wire x1="8.5725" y1="5.3975" x2="8.5725" y2="7.3025" width="0.254" layer="16"/>
@@
 <signal name="N$13">
 <contactref element="IC2" pad="5"/>
-<contactref element="ESP01" pad="TX"/>
+<contactref element="MOD1" pad="TX"/>
 <wire x1="7.9375" y1="5.715" x2="7.9375" y2="7.3025" width="0.254" layer="16"/>
 <wire x1="13.335" y1="5.715" x2="7.9375" y2="5.715" width="0.254" layer="1"/>
@@
 <signal name="N$14">
 <contactref element="IC2" pad="6"/>
-<contactref element="ESP01" pad="CH_PD"/>
+<contactref element="MOD1" pad="CH_PD"/>
 <wire x1="7.3025" y1="5.08" x2="7.3025" y2="7.3025" width="0.254" layer="16"/>
 <wire x1="7.62" y1="4.7625" x2="7.3025" y2="5.08" width="0.254" layer="1"/>
