File: ESP_01_5V.sch (EAGLE design)
At the start: 12 parts, among them IC1 REG1117, IC2 IC_TXB0108-TSSOP-20

Commit message: update
Parts:
- removed ESP01: ESP01, esp8266modules:ESP01
- added MOD1: ESP01, esp8266modules:ESP01
Connections:
- net 3.3V: now also MOD1.VCC; no longer ESP01.VCC
- net GND: now also MOD1.GND; no longer ESP01.GND
- net N$10: now also MOD1.RXD; no longer ESP01.RXD
- net N$11: now also MOD1.GPIO2; no longer ESP01.GPIO2
- net N$12: now also MOD1.GPIO0; no longer ESP01.GPIO0
- net N$13: now also MOD1.TXD; no longer ESP01.TXD
- net N$14: now also MOD1.CH_PD; no longer ESP01.CH_PD
- net N$9: now also MOD1.RST; no longer ESP01.RST
Other:
- note added: "https://github.com/sfranzyshen/ESP_01_5V"
- moved on the sheet: C1, C2, C3, C4, C5, C6, IC1, IC2, JP1, JP2, JP3
